File: hardware/PGTNX08_pitch_out.brd (EAGLE design)
At the start: 112.1 x 77.5 mm, 94 parts, among them IC1 AD420, IC10 AD420, IC11 AD420, IC2 AD420, IC3 AD420, IC4 TL084P, IC5 TL084P, IC6 AD420, IC7 AD420, IC9 AD420

Commit message: Tidy up scheamtics
Parts:
- added CLOCK2, DOUT, LATCH2: HEADER/MALE/01, connectors:HEADER/MALE/01
Connections:
- net N$37: now also CLOCK2.1
- net N$53: now also DOUT.1
- net N$69: now also LATCH2.1
Routing:
- net N$69: track 161.1 -> 161.7 mm
Other:
- board text added: "ANALOG OUTPUTS"
- board text added: "INPUTS"
- board text added: "OUTPUTS"
