File: hardware/PGTNX08_pitch_out.sch (EAGLE design)
At the start: 89 parts, among them IC1 AD420, IC10 AD420, IC11 AD420, IC2 AD420, IC3 AD420, IC4 TL084P, IC5 TL084P, IC6 AD420, IC7 AD420, IC9 AD420

Commit message: Tidy up scheamtics
Parts:
- added CLOCK2, DOUT, LATCH2: HEADER/MALE/01, connectors:HEADER/MALE/01
Connections:
- net N$37: now also CLOCK2.3
- net N$53: now also DOUT.3
- net N$69: now also LATCH2.3
