File: hardware/PGTNX07_gate_out.sch (EAGLE design)
At the start: 104 parts, among them IC1 74HC595N, IC10 74HC595N, IC11 TL074P, IC12 TL074P, IC2 TL074P, IC3 TL074P, IC4 74HC595N, IC5 TL074P, IC6 TL074P, IC7 74HC595N, IC8 TL074P, IC9 TL074P

Commit message: Tidy up scheamtics
Parts:
- added CLOCK2, LATCH2: HEADER/MALE/01, connectors:HEADER/MALE/01
Connections:
- net CLK2 renamed +5V
- net N$19: now also CLOCK2.3
- net N$33: now also LATCH2.3

Commit message: Added seperate headers for driving leds from outputs
Parts:
- added LED1, LED10, LED11, LED12, LED13, LED14, LED15, LED16, LED17, LED18, LED19, LED2, LED20, LED21, LED22, LED23, LED24, LED25, LED26, LED27, LED28, LED29, LED3, LED30, LED31, LED32, LED4, LED5, LED6, LED7, LED8, LED9: HEADER/MALE/01, connectors:HEADER/MALE/01
- renumbered OUT1 to 1, OUT10 to 10, OUT11 to 11, OUT12 to 12, OUT13 to 13, OUT14 to 14, OUT15 to 15, OUT16 to 16, OUT17 to 17, OUT18 to 18, OUT19 to 19, OUT2 to 2, OUT20 to 20, OUT21 to 21, OUT22 to 22, OUT23 to 23, OUT24 to 24, OUT25 to 25, OUT26 to 26, OUT27 to 27, OUT28 to 28, OUT29 to 29, OUT3 to 3, OUT30 to 30, OUT31 to 31, OUT32 to 32, OUT4 to 4, OUT5 to 5, OUT6 to 6, OUT7 to 7, OUT8 to 8, OUT9 to 9
Connections:
- net N$103: now also LED27.3
- net N$104: now also LED28.3
- net N$105: now also LED29.3
- net N$106: now also LED30.3
- net N$107: now also LED31.3
- net N$108: now also LED32.3
- net N$14: now also LED1.3
- net N$16: now also LED2.3
- net N$27: now also LED3.3
- net N$28: now also LED4.3
- net N$29: now also LED5.3
- net N$30: now also LED6.3
- net N$31: now also LED7.3
- net N$32: now also LED8.3
- net N$44: now also LED9.3
- net N$46: now also LED10.3
- net N$55: now also LED11.3
- net N$56: now also LED12.3
- net N$57: now also LED13.3
- net N$58: now also LED14.3
- net N$59: now also LED15.3
- net N$60: now also LED16.3
- net N$69: now also LED17.3
- net N$71: now also LED18.3
- net N$78: now also LED19.3
- net N$79: now also LED20.3
- net N$80: now also LED21.3
- net N$81: now also LED22.3
- net N$82: now also LED23.3
- net N$83: now also LED24.3
- net N$94: now also LED25.3
- net N$96: now also LED26.3
