File: hardware/PGTNX05_mainboard.brd (EAGLE design)
At the start: 111.8 x 77.5 mm, 180 parts, among them IC1 H11L1, IC2 LM2574N-5.0, IC3 40106N, IC4 H11L1

Commit message: Added correct diode type BZX55C12
Parts:
- D2, D3: value (none) -> BZX55C12
Changed lines of the file:
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@@
 <attribute name="VALUE" x="46.101" y="24.0538" size="1.27" layer="27" ratio="10" rot="R180"/>
 </element>
-<element name="D2" library="transistors" package="DO35-7" value="" x="43.18" y="22.86" smashed="yes">
+<element name="D2" library="transistors" package="DO35-7" value="BZX55C12" x="43.18" y="22.86" smashed="yes">
 <attribute name="NAME" x="42.164" y="22.225" size="1.27" layer="25" ratio="10"/>
 <attribute name="VALUE" x="40.894" y="20.193" size="1.27" layer="27" ratio="10"/>
 </element>
-<element name="D3" library="transistors" package="DO35-7" value="" x="43.18" y="30.48" smashed="yes" rot="R180">
+<element name="D3" library="transistors" package="DO35-7" value="BZX55C12" x="43.18" y="30.48" smashed="yes" rot="R180">
 <attribute name="NAME" x="44.196" y="31.115" size="1.27" layer="25" ratio="10" rot="R180"/>
 <attribute name="VALUE" x="45.466" y="33.147" size="1.27" layer="27" ratio="10" rot="R180"/>

Commit message: Add resistor values
Parts:
- R1, R10, R11, R12, R13, R14, R15, R16, R17, R18, R19, R2, R20, R21, R22, R3, R4, R5, R6, R7, R8, R9: value (none) -> 1k
